Commit message: Parameterize robot model and synchronize simulation geometry
Introduce a validated robot design YAML for chassis, wheels, sensors, racket geometry, mass, primitive inertia and joint limits. Apply the same configuration to URDF, sensor poses, scan and camera models, racket contacts and swing timing. Enforce wheel speed limits and extend swing duration to respect configured velocity.

Add a non-default robot profile, configuration documentation, numerical consistency tests and a configured ROS smoke case. Validate in Foxy Docker (five packages, zero test failures, five smoke modes) and expand both robot profiles with Humble Xacro.

File: packages/robom1_description/urdf/robom1.urdf.xacro (robot description, xacro)
@@ -1,90 +1,96 @@
 <?xml version="1.0"?>
 <robot xmlns:xacro="http://www.ros.org/wiki/xacro" name="robom1">
-  <xacro:arg name="wheelbase" default="0.52"/>
-  <xacro:arg name="track" default="0.48"/>
-  <xacro:arg name="wheel_radius" default="0.09"/>
-  <xacro:arg name="racket_pivot_x" default="0.05"/>
-  <xacro:property name="racket_pivot_x" value="$(arg racket_pivot_x)"/>
-  <xacro:arg name="racket_pivot_y" default="-0.36"/>
-  <xacro:property name="racket_pivot_y" value="$(arg racket_pivot_y)"/>
-  <xacro:arg name="racket_pivot_z" default="1.05"/>
-  <xacro:property name="racket_pivot_z" value="$(arg racket_pivot_z)"/>
-  <xacro:arg name="racket_reach" default="0.62"/>
-  <xacro:property name="racket_reach" value="$(arg racket_reach)"/>
-  <xacro:arg name="racket_radius" default="0.14"/>
-  <xacro:property name="racket_radius" value="$(arg racket_radius)"/>
-  <xacro:arg name="racket_thickness" default="0.015"/>
-  <xacro:property name="racket_thickness" value="$(arg racket_thickness)"/>
-  <xacro:property name="wb" value="$(arg wheelbase)"/>
-  <xacro:property name="tw" value="$(arg track)"/>
-  <xacro:property name="wr" value="$(arg wheel_radius)"/>
+  <xacro:arg name="robot_config" default="$(find robom1_description)/config/robot.yaml"/>
+  <xacro:property name="cfg" value="${load_yaml('$(arg robot_config)')}"/>
+  <xacro:property name="body" value="${cfg['chassis']}"/>
+  <xacro:property name="wh" value="${cfg['wheels']}"/>
+  <xacro:property name="mast" value="${cfg['mast']}"/>
+  <xacro:property name="cam" value="${cfg['camera']}"/>
+  <xacro:property name="lid" value="${cfg['lidar']}"/>
+  <xacro:property name="rac" value="${cfg['racket']}"/>
   <material name="blue"><color rgba="0.08 0.3 0.8 1"/></material>
   <material name="black"><color rgba="0.08 0.08 0.1 1"/></material>
   <material name="silver"><color rgba="0.7 0.75 0.8 1"/></material>
   <material name="orange"><color rgba="1 0.4 0.05 1"/></material>
-  <xacro:macro name="box_inertia" params="mass x y z">
-    <inertial><mass value="${mass}"/><inertia ixx="${mass*(y*y+z*z)/12}" ixy="0" ixz="0"
-      iyy="${mass*(x*x+z*z)/12}" iyz="0" izz="${mass*(x*x+y*y)/12}"/></inertial>
+  <!-- Solid primitive approximations; mass is per link. Inertia is about its COM. -->
+  <xacro:macro name="box_inertia" params="mass x y z cz:=0.0">
+    <inertial><origin xyz="0 0 ${cz}"/><mass value="${mass}"/>
+      <inertia ixx="${mass*(y*y+z*z)/12}" ixy="0" ixz="0"
+        iyy="${mass*(x*x+z*z)/12}" iyz="0" izz="${mass*(x*x+y*y)/12}"/></inertial>
+  </xacro:macro>
+  <xacro:macro name="cylinder_inertia" params="mass radius length axis">
+    <xacro:property name="axial" value="${mass*radius*radius/2}"/>
+    <xacro:property name="transverse" value="${mass*(3*radius*radius+length*length)/12}"/>
+    <inertial><mass value="${mass}"/><inertia
+      ixx="${axial if axis == 'x' else transverse}" ixy="0" ixz="0"
+      iyy="${axial if axis == 'y' else transverse}" iyz="0" izz="${transverse}"/></inertial>
   </xacro:macro>
   <xacro:macro name="box_link" params="name size mass color">
     <link name="${name}">
-      <visual><geometry><box size="${size}"/></geometry><material name="${color}"/></visual>
-      <collision><geometry><box size="${size}"/></geometry></collision>
-      <xacro:box_inertia mass="${mass}" x="${float(size.split()[0])}" y="${float(size.split()[1])}" z="${float(size.split()[2])}"/>
+      <visual><geometry><box size="${size[0]} ${size[1]} ${size[2]}"/></geometry><material name="${color}"/></visual>
+      <collision><geometry><box size="${size[0]} ${size[1]} ${size[2]}"/></geometry></collision>
+      <xacro:box_inertia mass="${mass}" x="${size[0]}" y="${size[1]}" z="${size[2]}"/>
     </link>
   </xacro:macro>
+  <xacro:macro name="mount_origin" params="xyz rpy">
+    <origin xyz="${xyz[0]} ${xyz[1]} ${xyz[2]-body['center_z']}" rpy="${rpy[0]} ${rpy[1]} ${rpy[2]}"/>
+  </xacro:macro>
   <link name="base_footprint"/>
-  <xacro:box_link name="base_link" size="0.64 0.44 0.16" mass="18.0" color="blue"/>
-  <joint name="base_joint" type="fixed"><parent link="base_footprint"/><child link="base_link"/><origin xyz="0 0 0.22"/></joint>
-  <xacro:macro name="wheel" params="name x y">
-    <xacro:box_link name="${name}_steer_link" size="0.06 0.06 0.06" mass="0.3" color="orange"/>
-    <joint name="${name}_steer_joint" type="continuous">
-      <parent link="base_link"/><child link="${name}_steer_link"/>
-      <origin xyz="${x} ${y} ${wr-0.22}"/><axis xyz="0 0 1"/><limit effort="20" velocity="4"/>
+  <xacro:box_link name="base_link" size="${body['size']}" mass="${body['mass']}" color="blue"/>
+  <joint name="base_joint" type="fixed"><parent link="base_footprint"/><child link="base_link"/>
+    <origin xyz="0 0 ${body['center_z']}"/></joint>
+  <xacro:macro name="wheel_module" params="name x y">
+    <xacro:box_link name="${name}_steer_link" size="${wh['steer_size']}" mass="${wh['steer_mass']}" color="orange"/>
+    <joint name="${name}_steer_joint" type="continuous"><parent link="base_link"/><child link="${name}_steer_link"/>
+      <origin xyz="${x} ${y} ${wh['radius']-body['center_z']}"/><axis xyz="0 0 1"/>
+      <limit effort="${wh['steer_effort']}" velocity="${wh['steer_velocity']}"/>
+      <dynamics damping="${wh['damping']}" friction="${wh['friction']}"/>
     </joint>
     <link name="${name}_wheel_link">
-      <visual><origin rpy="${pi/2} 0 0"/><geometry><cylinder radius="${wr}" length="0.045"/></geometry><material name="black"/></visual>
-      <collision><origin rpy="${pi/2} 0 0"/><geometry><cylinder radius="${wr}" length="0.045"/></geometry></collision>
-      <inertial><mass value="0.5"/><inertia ixx="${0.5*(3*wr*wr+0.045*0.045)/12}" ixy="0" ixz="0"
-        iyy="${0.5*wr*wr/2}" iyz="0" izz="${0.5*(3*wr*wr+0.045*0.045)/12}"/></inertial>
+      <visual><origin rpy="${pi/2} 0 0"/><geometry><cylinder radius="${wh['radius']}" length="${wh['width']}"/></geometry><material name="black"/></visual>
+      <collision><origin rpy="${pi/2} 0 0"/><geometry><cylinder radius="${wh['radius']}" length="${wh['width']}"/></geometry></collision>
+      <xacro:cylinder_inertia mass="${wh['mass']}" radius="${wh['radius']}" length="${wh['width']}" axis="y"/>
     </link>
-    <joint name="${name}_wheel_joint" type="continuous"><parent link="${name}_steer_link"/>
-      <child link="${name}_wheel_link"/><axis xyz="0 1 0"/><limit effort="20" velocity="40"/></joint>
+    <joint name="${name}_wheel_joint" type="continuous"><parent link="${name}_steer_link"/><child link="${name}_wheel_link"/>
+      <axis xyz="0 1 0"/><limit effort="${wh['drive_effort']}" velocity="${wh['drive_velocity']}"/>
+      <dynamics damping="${wh['damping']}" friction="${wh['friction']}"/>
+    </joint>
   </xacro:macro>
-  <xacro:wheel name="front_left" x="${wb/2}" y="${tw/2}"/>
-  <xacro:wheel name="front_right" x="${wb/2}" y="${-tw/2}"/>
-  <xacro:wheel name="rear_left" x="${-wb/2}" y="${tw/2}"/>
-  <xacro:wheel name="rear_right" x="${-wb/2}" y="${-tw/2}"/>
-  <xacro:box_link name="mast_link" size="0.05 0.05 0.7" mass="1.0" color="silver"/>
-  <joint name="mast_joint" type="fixed"><parent link="base_link"/><child link="mast_link"/><origin xyz="0 0 0.43"/></joint>
-  <!-- Absolute sensor positions: camera (0.12,0,1.0), lidar (0.18,0,0.90). -->
-  <xacro:box_link name="camera_link" size="0.06 0.10 0.04" mass="0.1" color="black"/>
-  <joint name="camera_joint" type="fixed"><parent link="base_link"/><child link="camera_link"/><origin xyz="0.12 0 0.78"/></joint>
+  <xacro:wheel_module name="front_left" x="${wh['wheelbase']/2}" y="${wh['track']/2}"/>
+  <xacro:wheel_module name="front_right" x="${wh['wheelbase']/2}" y="${-wh['track']/2}"/>
+  <xacro:wheel_module name="rear_left" x="${-wh['wheelbase']/2}" y="${wh['track']/2}"/>
+  <xacro:wheel_module name="rear_right" x="${-wh['wheelbase']/2}" y="${-wh['track']/2}"/>
+  <xacro:box_link name="mast_link" size="${mast['size']}" mass="${mast['mass']}" color="silver"/>
+  <joint name="mast_joint" type="fixed"><parent link="base_link"/><child link="mast_link"/>
+    <xacro:mount_origin xyz="${mast['xyz']}" rpy="${[0,0,0]}"/></joint>
+  <xacro:box_link name="camera_link" size="${cam['size']}" mass="${cam['mass']}" color="black"/>
+  <joint name="camera_joint" type="fixed"><parent link="base_link"/><child link="camera_link"/>
+    <xacro:mount_origin xyz="${cam['xyz']}" rpy="${cam['rpy']}"/></joint>
   <link name="camera_optical_frame"/>
-  <joint name="camera_optical_joint" type="fixed"><parent link="camera_link"/><child link="camera_optical_frame"/><origin rpy="${-pi/2} 0 ${-pi/2}"/></joint>
-  <xacro:box_link name="lidar_link" size="0.07 0.07 0.06" mass="0.2" color="orange"/>
-  <!-- Positive pitch raises the beam: rotation about NEGATIVE y. -->
+  <joint name="camera_optical_joint" type="fixed"><parent link="camera_link"/><child link="camera_optical_frame"/>
+    <origin rpy="${-pi/2} 0 ${-pi/2}"/></joint>
+  <xacro:box_link name="lidar_link" size="${lid['size']}" mass="${lid['mass']}" color="orange"/>
   <joint name="lidar_pitch_joint" type="revolute"><parent link="base_link"/><child link="lidar_link"/>
-    <origin xyz="0.18 0 0.68"/><axis xyz="0 -1 0"/>
-    <limit lower="-0.6" upper="1.2" effort="4" velocity="1.5"/>
+    <xacro:mount_origin xyz="${lid['xyz']}" rpy="${lid['rpy']}"/><axis xyz="0 -1 0"/>
+    <limit lower="${lid['lower']}" upper="${lid['upper']}" effort="${lid['effort']}" velocity="${lid['velocity']}"/>
+    <dynamics damping="${lid['damping']}" friction="${lid['friction']}"/>
   </joint>
-  <!-- Grip-end pivot: local +z points from grip to head. Positive +y pitch
-       sweeps the head forward (+x), then down through the follow-through. -->
   <link name="racket_handle_link">
-    <visual><origin xyz="0 0 0.25"/><geometry><box size="0.025 0.025 0.5"/></geometry><material name="silver"/></visual>
-    <visual><origin xyz="0 0 0.06"/><geometry><box size="0.04 0.04 0.12"/></geometry><material name="black"/></visual>
-    <collision><origin xyz="0 0 0.25"/><geometry><box size="0.025 0.025 0.5"/></geometry></collision>
-    <inertial><origin xyz="0 0 0.25"/><mass value="0.1"/>
-      <inertia ixx="0.00208854" ixy="0" ixz="0" iyy="0.00208854" iyz="0" izz="0.00001042"/></inertial>
+    <visual><origin xyz="0 0 ${rac['handle_length']/2}"/><geometry><box size="${rac['handle_width']} ${rac['handle_width']} ${rac['handle_length']}"/></geometry><material name="silver"/></visual>
+    <visual><origin xyz="0 0 ${rac['grip_length']/2}"/><geometry><box size="${rac['grip_width']} ${rac['grip_width']} ${rac['grip_length']}"/></geometry><material name="black"/></visual>
+    <collision><origin xyz="0 0 ${rac['handle_length']/2}"/><geometry><box size="${rac['handle_width']} ${rac['handle_width']} ${rac['handle_length']}"/></geometry></collision>
+    <xacro:box_inertia mass="${rac['handle_mass']}" x="${rac['handle_width']}" y="${rac['handle_width']}" z="${rac['handle_length']}" cz="${rac['handle_length']/2}"/>
   </link>
   <joint name="racket_swing_joint" type="revolute"><parent link="base_link"/><child link="racket_handle_link"/>
-    <origin xyz="${racket_pivot_x} ${racket_pivot_y} ${float(racket_pivot_z)-0.22}"/><axis xyz="0 1 0"/>
-    <limit lower="-1.8" upper="2.0" effort="10" velocity="8"/>
+    <xacro:mount_origin xyz="${rac['pivot']}" rpy="${rac['rpy']}"/><axis xyz="0 1 0"/>
+    <limit lower="${rac['lower']}" upper="${rac['upper']}" effort="${rac['effort']}" velocity="${rac['velocity']}"/>
+    <dynamics damping="${rac['damping']}" friction="${rac['friction']}"/>
   </joint>
   <link name="racket_head_link">
-    <visual><origin rpy="0 ${pi/2} 0"/><geometry><cylinder radius="${racket_radius}" length="${racket_thickness}"/></geometry><material name="orange"/></visual>
-    <collision><origin rpy="0 ${pi/2} 0"/><geometry><cylinder radius="${racket_radius}" length="${racket_thickness}"/></geometry></collision>
-    <xacro:box_inertia mass="0.08" x="${racket_thickness}" y="${2*float(racket_radius)}" z="${2*float(racket_radius)}"/>
+    <visual><origin rpy="0 ${pi/2} 0"/><geometry><cylinder radius="${rac['radius']}" length="${rac['thickness']}"/></geometry><material name="orange"/></visual>
+    <collision><origin rpy="0 ${pi/2} 0"/><geometry><cylinder radius="${rac['radius']}" length="${rac['thickness']}"/></geometry></collision>
+    <xacro:cylinder_inertia mass="${rac['head_mass']}" radius="${rac['radius']}" length="${rac['thickness']}" axis="x"/>
   </link>
-  <joint name="racket_head_joint" type="fixed"><parent link="racket_handle_link"/><child link="racket_head_link"/><origin xyz="0 0 ${racket_reach}"/></joint>
+  <joint name="racket_head_joint" type="fixed"><parent link="racket_handle_link"/><child link="racket_head_link"/>
+    <origin xyz="0 0 ${rac['reach']}"/></joint>
 </robot>
